Commit message: Update URDF to use meshes

File: mobile_robot_description/urdf/mobile_robot.urdf (robot description, URDF)
Before this commit: robot mobilerobot, 6 links, 5 joints
Links:
- link base_link: geometry collision box size=0.13 0.1 0.078; visual box size=0.005 0.065 0.02
- link caster_support: geometry collision box size=0.04 0.009 0.025; visual mesh filename=package://mobile_robot_description/meshes/mobile_robot_cast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

Commit message: Make displayable in Gazebo

File: mobile_robot_description/urdf/mobile_robot.urdf (robot description, URDF)
Before this commit: robot mobilerobot, 6 links, 5 joints
Links:
- link base_link: mass None -> 0.25
- link caster_support: mass None -> 0.1
- link caster_wheel: mass None -> 0.1
- link laser: mass None -> 0.6
- link left_wheel: mass None -> 0.1
- link right_wheel: mass None -> 0.1
