Commit message: Add Gazebo info

File: manipulator_description/urdf/manipulator.urdf.xacro (robot description, xacro)
@@ -27,3 +27,18 @@
       base_colour="black"
       finger_colour="grey"/>
+  <!-- Include Gazebo-specific information if in simulation mode -->
+  <xacro:if value="$(arg use_simulation)">
+    <xacro:include filename="$(find manipulator_description)/urdf/manipulator.gazebo.xacro"/>
+    <xacro:basic_transmission joint_name="shoulder_rotate_joint"/>
+    <xacro:basic_transmission joint_name="shoulder_pitch_joint"/>
+    <xacro:basic_transmission joint_name="upper_arm_link_joint"/>
+    <xacro:basic_transmission joint_name="lower_arm_link_joint"/>
+    <xacro:basic_transmission joint_name="moving_finger_joint"/>
+    <gazebo>
+      <plugin name="control" filename="libgazebo_ros_control.so"/>
+      <plugin name="joint_state_publisher" filename="libgazebo_ros_joint_state_publisher.so">
+        <jointName>shoulder_rotate_joint, shoulder_pitch_joint, upper_arm_link_joint, lower_arm_link_joint, moving_finger_joint</jointName>
+      </plugin>
+    </gazebo>
+  </xacro:if>
 </robot>

File: manipulator_description/urdf/manipulator_parts.xacro (robot description, xacro)
@@ -35,5 +35,5 @@
     </link>
     <!-- Joint to rotate the shoulder about the Z axis (yaw) -->
-    <joint name="shoulder_rotate" type="revolute">
+    <joint name="shoulder_rotate_joint" type="revolute">
       <axis xyz="0 0 1"/>
       <parent link="base_link"/>
@@ -80,5 +80,5 @@
     </link>
     <!-- Joint to rotate the shoulder about the Y axis (pitch) -->
-    <joint name="shoulder_pitch" type="revolute">
+    <joint name="shoulder_pitch_joint" type="revolute">
       <axis xyz="0 1 0"/>
       <parent link="shoulder_link"/>
