Commit message: For visualising the CRANE+ hardware

File: manipulator_description/urdf/manipulator_parts.xacro (robot description, xacro)
@@ -35,5 +35,5 @@
     </link>
     <!-- Joint to rotate the shoulder about the Z axis (yaw) -->
-    <joint name="shoulder_rotate_joint" type="revolute">
+    <joint name="crane_plus_shoulder_revolute_joint" type="revolute">
       <axis xyz="0 0 1"/>
       <parent link="base_link"/>
@@ -80,14 +80,14 @@
     </link>
     <!-- Joint to rotate the shoulder about the Y axis (pitch) -->
-    <joint name="shoulder_pitch_joint" type="revolute">
+    <joint name="crane_plus_shoulder_flex_joint" type="revolute">
       <axis xyz="0 1 0"/>
       <parent link="shoulder_link"/>
-      <child link="upper_arm_link"/>
+      <child link="crane_plus_elbow"/>
       <origin xyz="0 0 ${SHOULDER_Z-0.01}" rpy="0 0 0"/>
       <limit lower="-${PI}" upper="${PI}" effort="30" velocity="${PI}"/>
     </joint>
     <!-- Upper arm link and joint -->
-    <xacro:arm_link link_name="upper_arm_link"
-        child_link_name="lower_arm_link"
+    <xacro:arm_link link_name="crane_plus_elbow"
+        child_link_name="crane_plus_wrist"
         llimit="-${2 * PI / 3}"
         ulimit="${2 * PI / 3}"
@@ -96,5 +96,5 @@
     <!-- The far joint of this link is connected to the externally-specific link, which is usually
          an end effector. -->
-    <xacro:arm_link link_name="lower_arm_link"
+    <xacro:arm_link link_name="crane_plus_wrist"
         child_link_name="${end_effector_link}"
         llimit="${-2 * PI / 3}"

File: manipulator_description/urdf/one_finger_gripper.xacro (robot description, xacro)
@@ -87,5 +87,5 @@
     </link>
     <!-- Revolute joint to moving finger -->
-    <joint name="moving_finger_joint" type="revolute">
+    <joint name="crane_plus_moving_finger_joint" type="revolute">
       <axis xyz="1 0 0"/>
       <parent link="${base_link_name}"/>

Commit message: Reverse joint axes to match real hardware

File: manipulator_description/urdf/manipulator_parts.xacro (robot description, xacro)
@@ -92,4 +92,5 @@
         llimit="-${2 * PI / 3}"
         ulimit="${2 * PI / 3}"
+        orientation="-1"
         colour="${link_colour_1}"/>
     <!-- Lower arm link and joint -->
@@ -100,4 +101,5 @@
         llimit="${-2 * PI / 3}"
         ulimit="${2 * PI / 3}"
+        orientation="-1"
         colour="${link_colour_2}"/>
   </xacro:macro>
@@ -105,5 +107,5 @@
   <!-- *origin parameter is for the joint at the child end of the link, not for where this link is
        rooted -->
-  <xacro:macro name="arm_link" params="link_name child_link_name llimit ulimit colour">
+  <xacro:macro name="arm_link" params="link_name child_link_name llimit ulimit orientation:=1 colour">
     <xacro:property name="ARM_LINK_X" value="0.032"/>
     <xacro:property name="ARM_LINK_Y" value="0.038"/>
@@ -130,5 +132,5 @@
     <!-- This joint joins to the specified child link -->
     <joint name="${link_name}_joint" type="revolute">
-      <axis xyz="0 1 0"/>
+      <axis xyz="0 ${orientation} 0"/>
       <parent link="${link_name}"/>
       <child link="${child_link_name}"/>
